File: Motors1-4.sch (KiCad schematic (older format))
At the start: 23 parts

Commit message: Component Placement.
Parts:
- C201, C202: renamed from C?; footprint (none) -> Capacitors_SMD:C_0603_HandSoldering
- J201, J202, J203, J204: renamed from J?; footprint (none) -> Terminal_Blocks:TerminalBlock_Pheonix_MPT-2.54mm_5pol
- U201, U202, U203, U204: renamed from U?; footprint (none) -> Housings_SOIC:SOIC-8_3.9x4.9mm_Pitch1.27mm
- U205, U206: renamed from U?; footprint (none) -> Housings_SOIC:SOIC-14_3.9x8.7mm_Pitch1.27mm
- gave numbers to parts that had none: 1

Commit message: Component Placement.
Parts:
- removed RN201: 10K, Resistors_THT:R_Array_SIP9, symbol R_Network08
- added R201, R202, R203, R204, R205, R206, R207, R208: 10K, Resistors_SMD:R_0603_HandSoldering, symbol R
Connections:
- net +3V3: now also R201.1, R202.2, R203.1, R204.2, R205.1, R206.2, R207.1, R208.2
- net P1A: now also R201.2
- net P1B: now also R202.1
- net P2A: now also R203.2
- net P2B: now also R204.1
- net P3A: now also R205.2
- net P3B: now also R206.1
- net P4A: now also R207.2
- net P4B: now also R208.1
