File: Motors5-8.sch (KiCad schematic (older format))
At the start: 23 parts

Commit message: Component Placement.
Parts:
- C301, C302: renamed from C?; footprint (none) -> Capacitors_SMD:C_0603_HandSoldering
- J301, J302, J303, J304: renamed from J?; footprint (none) -> Terminal_Blocks:TerminalBlock_Pheonix_MPT-2.54mm_5pol
- U301, U302, U303, U304: renamed from U?; footprint (none) -> Housings_SOIC:SOIC-8_3.9x4.9mm_Pitch1.27mm
- U305, U306: renamed from U?; footprint (none) -> Housings_SOIC:SOIC-14_3.9x8.7mm_Pitch1.27mm
- gave numbers to parts that had none: 1
Connections:
- net M5B: now also U301.5 (Out); no longer U301.7 (Out)
- net M6B: now also U302.5 (Out); no longer U302.7 (Out)
- net M7B: now also U303.5 (Out); no longer U303.7 (Out)
- net M8B: now also U304.5 (Out); no longer U304.7 (Out)
- net Motor5: now also U301.4 (IN); no longer U301.2 (IN)
- net Motor6: now also U302.4 (IN); no longer U302.2 (IN)
- net Motor7: now also U303.4 (IN); no longer U303.2 (IN)
- net Motor8: now also U304.4 (IN); no longer U304.2 (IN)
- net P5B: now also U305.5; no longer U305.2
- net P6A: now also U305.9; no longer U305.1
- net P6B: now also U305.13; no longer U305.2
- net P7B: now also U306.5; no longer U306.2
- net P8A: now also U306.9; no longer U306.1
- net P8B: now also U306.13; no longer U306.2
- net Points5: now also U305.4; no longer U305.1
- net Points6: now also U305.12, U305.8; no longer U305.1, U305.3
- net Points7: now also U306.4; no longer U306.1
- net Points8: now also U306.12, U306.8; no longer U306.1, U306.3
- net at U305.2: now also U305.6; no longer U305.3
- net at U306.2: now also U306.6; no longer U306.3
- new net: U305.10, U305.11
- new net: U306.10, U306.11

Commit message: Component Placement.
Parts:
- removed RN301: 10K, Resistors_THT:R_Array_SIP9, symbol R_Network08
- added R301, R302, R303, R304, R305, R306, R307, R308: 10K, Resistors_SMD:R_0603_HandSoldering, symbol R
Connections:
- net +3V3: now also R301.1, R302.2, R303.1, R304.2, R305.1, R306.2, R307.1, R308.2
- net P5A: now also R301.2
- net P5B: now also R302.1
- net P6A: now also R303.2
- net P6B: now also R304.1
- net P7A: now also R305.2
- net P7B: now also R306.1
- net P8A: now also R307.2
- net P8B: now also R308.1
