File: Esp32OlcbIO-8StallMotor.kicad_pcb (KiCad board)
At the start: 2 copper layers, 61 x 81 mm, 2 parts, among them J2 LEFT-EXT, J4 RIGHT-EXT

Commit message: Component Placement.
Parts:
- added C201: .1uf, Capacitors_SMD:C_0603_HandSoldering, F.Cu at (141.6, 68.3)
- added C202: .1uf, Capacitors_SMD:C_0603_HandSoldering, F.Cu at (143.2, 57.1)
- added C301: .1uf, Capacitors_SMD:C_0603_HandSoldering, F.Cu at (141.0, 80.3)
- added C302: .1uf, Capacitors_SMD:C_0603_HandSoldering, F.Cu at (141.6, 91.8)
- added J201: Motor 1, Terminal_Blocks:TerminalBlock_Pheonix_MPT-2.54mm_5pol, F.Cu at (161.9, 64.8)
- added J202: Motor 2, Terminal_Blocks:TerminalBlock_Pheonix_MPT-2.54mm_5pol, F.Cu at (161.9, 80.0)
- added J203: Motor 3, Terminal_Blocks:TerminalBlock_Pheonix_MPT-2.54mm_5pol, F.Cu at (161.9, 94.6)
- added J204: Motor 4, Terminal_Blocks:TerminalBlock_Pheonix_MPT-2.54mm_5pol, F.Cu at (161.9, 109.9)
- added J301: Motor 5, Terminal_Blocks:TerminalBlock_Pheonix_MPT-2.54mm_5pol, F.Cu at (111.8, 54.0)
- added J302: Motor 6, Terminal_Blocks:TerminalBlock_Pheonix_MPT-2.54mm_5pol, F.Cu at (111.8, 69.8)
- added J303: Motor 7, Terminal_Blocks:TerminalBlock_Pheonix_MPT-2.54mm_5pol, F.Cu at (111.8, 85.1)
- added J304: Motor 8, Terminal_Blocks:TerminalBlock_Pheonix_MPT-2.54mm_5pol, F.Cu at (111.8, 100.3)
- added RN201: 10K, Resistors_THT:R_Array_SIP9, F.Cu at (156.8, 68.6)
- added RN301: 10K, Resistors_THT:R_Array_SIP9, F.Cu at (116.8, 69.8)
- added U201: TC4428, Housings_SOIC:SOIC-8_3.9x4.9mm_Pitch1.27mm, F.Cu at (146.8, 66.7)
- added U202: TC4428, Housings_SOIC:SOIC-8_3.9x4.9mm_Pitch1.27mm, F.Cu at (146.8, 73.0)
- added U203: TC4428, Housings_SOIC:SOIC-8_3.9x4.9mm_Pitch1.27mm, F.Cu at (146.8, 79.4)
- added U204: TC4428, Housings_SOIC:SOIC-8_3.9x4.9mm_Pitch1.27mm, F.Cu at (146.8, 85.7)
- added U205: 74HC00, Housings_SOIC:SOIC-14_3.9x8.7mm_Pitch1.27mm, F.Cu at (136.7, 61.6)
- added U206: 74HC00, Housings_SOIC:SOIC-14_3.9x8.7mm_Pitch1.27mm, F.Cu at (136.7, 71.8)
- added U301: TC4428, Housings_SOIC:SOIC-8_3.9x4.9mm_Pitch1.27mm, F.Cu at (126.8, 61.0)
- added U302: TC4428, Housings_SOIC:SOIC-8_3.9x4.9mm_Pitch1.27mm, F.Cu at (126.8, 68.6)
- added U303: TC4428, Housings_SOIC:SOIC-8_3.9x4.9mm_Pitch1.27mm, F.Cu at (126.8, 75.6)
- added U304: TC4428, Housings_SOIC:SOIC-8_3.9x4.9mm_Pitch1.27mm, F.Cu at (126.8, 83.2)
- added U305: 74HC00, Housings_SOIC:SOIC-14_3.9x8.7mm_Pitch1.27mm, F.Cu at (135.1, 83.2)
- added U306: 74HC00, Housings_SOIC:SOIC-14_3.9x8.7mm_Pitch1.27mm, F.Cu at (135.7, 94.6)
Connections:
- J4 pad 1: VCC -> +VDC
Routing:
- added copper zone on F.Cu, net +3V3
- added copper zone on B.Cu, net GND

Commit message: Component Placement.
Parts:
- removed RN201, RN301: 10K, Resistors_THT:R_Array_SIP9
- added R201: 10K, Resistors_SMD:R_0603_HandSoldering, F.Cu at (157.5, 62.0)
- added R202: 10K, Resistors_SMD:R_0603_HandSoldering, F.Cu at (157.5, 53.3)
- added R203: 10K, Resistors_SMD:R_0603_HandSoldering, F.Cu at (157.5, 76.0)
- added R204: 10K, Resistors_SMD:R_0603_HandSoldering, F.Cu at (157.5, 69.0)
- added R205: 10K, Resistors_SMD:R_0603_HandSoldering, F.Cu at (157.5, 90.8)
- added R206: 10K, Resistors_SMD:R_0603_HandSoldering, F.Cu at (157.5, 83.7)
- added R207: 10K, Resistors_SMD:R_0603_HandSoldering, F.Cu at (157.5, 105.7)
- added R208: 10K, Resistors_SMD:R_0603_HandSoldering, F.Cu at (157.5, 98.5)
- added R301: 10K, Resistors_SMD:R_0603_HandSoldering, F.Cu at (116.3, 57.8)
- added R302: 10K, Resistors_SMD:R_0603_HandSoldering, F.Cu at (116.3, 65.4)
- added R303: 10K, Resistors_SMD:R_0603_HandSoldering, F.Cu at (116.3, 74.1)
- added R304: 10K, Resistors_SMD:R_0603_HandSoldering, F.Cu at (116.3, 81.2)
- added R305: 10K, Resistors_SMD:R_0603_HandSoldering, F.Cu at (116.3, 89.3)
- added R306: 10K, Resistors_SMD:R_0603_HandSoldering, F.Cu at (116.3, 96.6)
- added R307: 10K, Resistors_SMD:R_0603_HandSoldering, F.Cu at (116.3, 104.1)
- added R308: 10K, Resistors_SMD:R_0603_HandSoldering, F.Cu at (116.3, 111.3)
- moved C202 6.67 mm to (136.5, 57.1), turned to 0 degrees
- moved U306 6.38 mm to (136.4, 101.0)
- moved C302 6.11 mm to (136.2, 94.6), turned to 180 degrees
- moved U305 5.24 mm to (136.4, 88.3)
- moved C301 5.02 mm to (136.2, 81.9), turned to 180 degrees
- moved C201 4.85 mm to (136.8, 69.2), turned to 180 degrees
- moved U206 3.82 mm to (136.4, 75.6)
- moved U205 1.93 mm to (136.4, 63.5)
Routing:
- net +VDC: track 0.00 -> 90.7 mm, vias 0 -> 2
- net /Motors 5 to 8/M8B: track 0.00 -> 35.6 mm, vias 0 -> 1
- net /Motors 5 to 8/M8A: track 0.00 -> 34.8 mm, vias 0 -> 1
- net /Motors 5 to 8/M5A: track 0.00 -> 28.2 mm, vias 0 -> 1
- net /Motors 5 to 8/M7B: track 0.00 -> 27.5 mm, vias 0 -> 1
- net /Motors 5 to 8/M7A: track 0.00 -> 26.5 mm, vias 0 -> 1
- net /Motors 5 to 8/M5B: track 0.00 -> 23.9 mm, vias 0 -> 1
- net /Motors 5 to 8/M6B: track 0.00 -> 19.2 mm, vias 0 -> 1
- net /Motors 5 to 8/M6A: track 0.00 -> 19.1 mm, vias 0 -> 1
- net IO11: track 0.00 -> 16.9 mm, vias 0 -> 1
- net IO10: track 0.00 -> 11.3 mm, vias 0 -> 1
- net IO9: track 0.00 -> 10.2 mm, vias 0 -> 1
- net /Motors 5 to 8/P7A: track 0.00 -> 6.92 mm, vias 0 -> 1
- net /Motors 5 to 8/P7B: track 0.00 -> 6.71 mm, vias 0 -> 1
- net /Motors 5 to 8/P6A: track 0.00 -> 6.65 mm, vias 0 -> 1
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
Commit message: Completed Board.
Parts:
- moved C201 0.90 mm to (136.2, 69.8)
- turned C202 to 180 degrees
- turned U205 to 0 degrees
- turned U206 to 0 degrees
Routing:
- net GND: track 4.36 -> 93.1 mm, vias 3 -> 15
- net /Motors 1 to 4/P4A: track 0.00 -> 52.2 mm, vias 0 -> 4
- net /Motors 1 to 4/P4B: track 0.00 -> 51.3 mm, vias 0 -> 3
- net IO16: track 0.00 -> 47.3 mm, vias 0 -> 2
- net /Motors 1 to 4/P3A: track 0.00 -> 46.3 mm, vias 0 -> 3
- net IO4: track 0.00 -> 45.4 mm, vias 0 -> 3
- net /Motors 5 to 8/P5B: track 6.22 -> 50.8 mm, vias 1 -> 4
- net /Motors 1 to 4/P3B: track 0.00 -> 44.5 mm, vias 0 -> 5
- net /Motors 5 to 8/P5A: track 5.96 -> 47.2 mm, vias 1 -> 3
- net /Motors 1 to 4/M4A: track 0.00 -> 41.0 mm, vias 0 -> 1
- net /Motors 5 to 8/P6A: track 6.65 -> 47.6 mm, vias 1 -> 2
- net /Motors 1 to 4/M4B: track 0.00 -> 40.7 mm, vias 0 -> 1
- net IO14: track 0.00 -> 40.1 mm, vias 0 -> 1
- net IO5: track 0.00 -> 39.2 mm, vias 0 -> 2
- net /Motors 1 to 4/P1B: track 0.00 -> 39.2 mm, vias 0 -> 3
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